File: board/board2/board2.kicad_sch (KiCad schematic)
At the start: 12 parts, among them J1 Conn_01x05_Female

Commit message: Update board2.kicad_sch
Parts:
- removed R7: 680Ω, symbol Device:R
- removed R8: 510Ω, symbol Device:R
Connections:
- net +5V: now also J?.3 (Pin_3); no longer C1.1, C2.1, J1.5 (Pin_5), J?.4 (Pin_4), R1.2, R3.2
- net at C1.2, J1.1 (Pin_1), R5.1: now also R3.2
- net at C2.2, J1.3 (Pin_3), R6.1: now also R1.2
- net at J?.2 (Pin_2): now also R2.2, R3.1; no longer R2.1
- net at J?.1 (Pin_1): now also R1.1, R4.2; no longer R4.1
- new net GND: C1.1, C2.1, J1.5 (Pin_5), J?.4 (Pin_4), R2.1, R4.1
Other:
- note added: "1 2 3 4"
- note added: "channel A channel B vcc gnd"
- note removed: "4 3 2 1"
- note removed: "gnd vcc channel B channel A"
- note removed: "x1 : dividing bridge PS 5V"

Commit message: v0.1 pcb
Parts:
- removed J1: Conn_01x05_Female, symbol Connector:Conn_01x05_Female
- added H1, H2, H3, H4: MountingHole, MountingHole:MountingHole_3.2mm_M3_DIN965, symbol Mechanical:MountingHole
- added J1: Conn_01x04_Female, Connector_JST:JST_XH_B4B-XH-A_1x04_P2.50mm_Vertical, symbol Connector:Conn_01x04_Female
- C1, C2: footprint (none) -> Capacitor_THT:CP_Radial_D4.0mm_P2.00mm
- J2: renamed from J?; footprint (none) -> Connector_JST:JST_XH_B4B-XH-A_1x04_P2.50mm_Vertical
- R1, R3: value 400Ω -> 1kΩ; footprint (none) -> Resistor_THT:R_Axial_DIN0309_L9.0mm_D3.2mm_P12.70mm_Horizontal
- R2, R4: value 600Ω -> 1800Ω; footprint (none) -> Resistor_THT:R_Axial_DIN0309_L9.0mm_D3.2mm_P12.70mm_Horizontal
- R5, R6: footprint (none) -> Resistor_THT:R_Axial_DIN0309_L9.0mm_D3.2mm_P12.70mm_Horizontal
Connections:
- net +5V: now also J1.3 (Pin_3)
- net GND: now also J1.4 (Pin_4)
- net at C1.2, R3.2, R5.1: now also J1.1 (Pin_1)
- net at C2.2, R1.2, R6.1: now also J1.2 (Pin_2)
- no-connect marks 1 -> 0
Other:
- note removed: "1 2 3 4 5"
- note removed: "channel B vcc channel A x gnd"
