File: electronics/stepper_driver/stepper_driver.kicad_pcb (KiCad board)
At the start: 2 copper layers, 62 x 105 mm, 17 parts, among them J1 Conn_01x04_Female, J2 Conn_01x05_Female, J3 Conn_01x04_Female, J4 Conn_01x05_Female, J5 Conn_01x04_Female, J6 Conn_01x05_Female, J7 Conn_01x04_Female, J8 Conn_01x04_Female, J9 Conn_01x04_Female, U1 ULN2003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

Commit message: update issue with board. clean code
Parts:
- moved H4 17.5 mm to (77.0, 27.0)
- moved H1 9.00 mm to (115.0, 27.0)
Connections:
- C1 pad 2: VCC -> +5V
- C2 pad 2: VCC -> +5V
- J1 pad 3: VCC -> +5V
- J2 pad 1: VCC -> Net-(J2-Pad1)
- J2 pad 5: Net-(J2-Pad5) -> +5V
- J3 pad 3: VCC -> +5V
- J4 pad 1: VCC -> Net-(J4-Pad1)
- J4 pad 5: Net-(J4-Pad5) -> +5V
- J5 pad 3: VCC -> +5V
- J6 pad 1: VCC -> Net-(J6-Pad1)
- J6 pad 5: Net-(J6-Pad5) -> +5V
- J7 pad 3: VCC -> +5V
- J8 pad 3: VCC -> +5V
- J9 pad 3: VCC -> +5V
- U1 pad 10: Net-(J4-Pad4) -> Net-(J4-Pad2)
- U1 pad 12: Net-(J4-Pad2) -> Net-(J4-Pad4)
- U1 pad 13: Net-(J2-Pad5) -> Net-(J2-Pad1)
- U1 pad 14: Net-(J2-Pad4) -> Net-(J2-Pad2)
- U1 pad 16: Net-(J2-Pad2) -> Net-(J2-Pad4)
- U1 pad 9: VCC -> +5V
- U2 pad 12: Net-(J6-Pad5) -> Net-(J6-Pad1)
- U2 pad 13: Net-(J6-Pad4) -> Net-(J6-Pad2)
- U2 pad 15: Net-(J6-Pad2) -> Net-(J6-Pad4)
- U2 pad 16: Net-(J4-Pad5) -> Net-(J4-Pad1)
- U2 pad 9: VCC -> +5V
Routing:
- net +5V: track 0.00 -> 272.5 mm
- net VCC: track 230.2 -> 0.00 mm
- net Net-(J4-Pad5): track 30.7 -> 0.00 mm
- net Net-(J2-Pad1): track 0.00 -> 16.8 mm
- net Net-(J4-Pad2): track 37.1 -> 20.4 mm
- net Net-(J6-Pad1): track 0.00 -> 16.0 mm
- net Net-(J2-Pad5): track 15.7 -> 0.00 mm
- net Net-(J6-Pad5): track 14.5 -> 0.00 mm
- net Net-(J6-Pad2): track 30.5 -> 16.0 mm
- net Net-(J4-Pad1): track 0.00 -> 13.6 mm
- net Net-(J2-Pad2): track 30.2 -> 16.8 mm
- net Net-(J6-Pad3): track 26.7 -> 16.0 mm
- net Net-(J4-Pad3): track 31.3 -> 20.8 mm
- net Net-(J2-Pad3): track 26.5 -> 16.9 mm
- net Net-(J6-Pad4): track 22.7 -> 16.1 mm
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Other:
- board size 62 x 105 mm -> 62 x 98 mm
