File: electronics/stepper_driver/stepper_driver.kicad_sch (KiCad schematic)
At the start: 17 parts, among them J1 Conn_01x04_Female, J2 Conn_01x05_Female, J3 Conn_01x04_Female, J4 Conn_01x05_Female, J5 Conn_01x04_Female, J6 Conn_01x05_Female, J7 Conn_01x04_Female, J8 Conn_01x04_Female, J9 Conn_01x04_Female, U1 ULN2003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

Commit message: update issue with board. clean code
Connections:
- net +5V: now also J2.5 (Pin_5), J4.5 (Pin_5), J6.5 (Pin_5); no longer J2.1 (Pin_1), J4.1 (Pin_1), J6.1 (Pin_1)
- net at J6.2 (Pin_2): now also U2.13 (O4); no longer U2.15 (O2)
- net at J6.4 (Pin_4): now also U2.15 (O2); no longer U2.13 (O4)
- net at U2.12 (O5): now also J6.1 (Pin_1); no longer J6.5 (Pin_5)
- net at J4.2 (Pin_2): now also U1.10 (O7); no longer U1.12 (O5)
- net at J4.4 (Pin_4): now also U1.12 (O5); no longer U1.10 (O7)
- net at U2.16 (O1): now also J4.1 (Pin_1); no longer J4.5 (Pin_5)
- net at J2.2 (Pin_2): now also U1.14 (O3); no longer U1.16 (O1)
- net at J2.4 (Pin_4): now also U1.16 (O1); no longer U1.14 (O3)
- net at U1.13 (O4): now also J2.1 (Pin_1); no longer J2.5 (Pin_5)
Changed lines of the file:
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@@
     (pin "1")
   )
-  (symbol (lib_id "Connector:Conn_01x05_Female") (at 114.808 107.188 0) (unit 1)
+  (symbol (lib_id "Connector:Conn_01x05_Female") (at 114.808 107.188 0) (mirror x) (unit 1)
     (in_bom yes) (on_board yes) (fields_autoplaced)
-    (property "Reference" "J6" (id 0) (at 115.5192 106.3533 0)
-      (effects (font (size 1.27 1.27)) (justify left))
-    )
-    (property "Value" "Conn_01x05_Female" (id 1) (at 115.5192 108.8902 0)
-      (effects (font (size 1.27 1.27)) (justify left))
-    )
+    (property "Reference" "J6" (id 0) (at 114.173 97.951 0))
+    (property "Value" "Conn_01x05_Female" (id 1) (at 114.173 100.4879 0))
     (property "Footprint" "Connector_JST:JST_XH_S5B-XH-A_1x05_P2.50mm_Horizontal" (id 2) (at 114.808 107.188 0)
       (effects (font (size 1.27 1.27)) hide)
@@
     (pin "1")
   )
-  (symbol (lib_id "Connector:Conn_01x05_Female") (at 114.808 89.662 0) (unit 1)
+  (symbol (lib_id "Connector:Conn_01x05_Female") (at 114.808 89.662 0) (mirror x) (unit 1)
     (in_bom yes) (on_board yes) (fields_autoplaced)
-    (property "Reference" "J4" (id 0) (at 115.5192 88.8273 0)
-      (effects (font (size 1.27 1.27)) (justify left))
-    )
-    (property "Value" "Conn_01x05_Female" (id 1) (at 115.5192 91.3642 0)
-      (effects (font (size 1.27 1.27)) (justify left))
-    )
+    (property "Reference" "J4" (id 0) (at 114.173 80.425 0))
+    (property "Value" "Conn_01x05_Female" (id 1) (at 114.173 82.9619 0))
     (property "Footprint" "Connector_JST:JST_XH_S5B-XH-A_1x05_P2.50mm_Horizontal" (id 2) (at 114.808 89.662 0)
       (effects (font (size 1.27 1.27)) hide)
@@
     (pin "4")
   )
-  (symbol (lib_id "Connector:Conn_01x05_Female") (at 114.3 70.612 0) (unit 1)
+  (symbol (lib_id "Connector:Conn_01x05_Female") (at 114.3 70.612 0) (mirror x) (unit 1)
     (in_bom yes) (on_board yes) (fields_autoplaced)
-    (property "Reference" "J2" (id 0) (at 115.0112 69.7773 0)
-      (effects (font (size 1.27 1.27)) (justify left))
-    )
-    (property "Value" "Conn_01x05_Female" (id 1) (at 115.0112 72.3142 0)
-      (effects (font (size 1.27 1.27)) (justify left))
-    )
+    (property "Reference" "J2" (id 0) (at 113.665 61.375 0))
+    (property "Value" "Conn_01x05_Female" (id 1) (at 113.665 63.9119 0))
     (property "Footprint" "Connector_JST:JST_XH_S5B-XH-A_1x05_P2.50mm_Horizontal" (id 2) (at 114.3 70.612 0)
       (effects (font (size 1.27 1.27)) hide)
